File: heepidermis-bo/heepidermis-bo.kicad_pcb (KiCad board)
At the start: 4 copper layers, 85.7 x 54 mm, 40 parts, among them J1 Conn_01x03, J10 Conn_Boaxial, J11 Conn_Boaxial, J12 Conn_01x03, J13 Conn_01x03, J14 Conn_01x03, J15 Conn_02x16_Odd_Even, J17 Conn_02x10_Odd_Even, J18 Conn_01x03, J19 Conn_01x03, J2 5025983393, J20 Conn_01x03, J21 Conn_01x03, J22 Conn_01x03, J23 Conn_02x29_Top_Bottom, J5 Conn_01x03, J6 Conn_01x03, J7 Conn_01x03, J8 Conn_01x03, J9 Conn_Boaxial, SW1 SW_Push

Commit message: DRC clean
Parts:
- removed the REF** at (109.7, 121.3)
- added G***: LOGO, LOGO, F.Cu at (107.9, 121.2)
- J23: footprint Connector_PinHeader_2.54mm:PinHeader_2x32_P2.54mm_Vertical -> Connector_PinHeader_2.54mm:PinHeader_2x32_P2.54mm_Horizontal
- R1, R2, R3: footprint X-MODs_PcbLib:R0402 -> Resistor_SMD:R_0402_1005Metric
- moved J8 3.72 mm to (141.6, 82.6)
- moved J6 2.83 mm to (113.3, 100.7), turned to -90 degrees
- moved J5 2.82 mm to (118.2, 100.7), turned to -90 degrees
- moved J12 1.34 mm to (170.3, 102.9)
- moved C1 1.23 mm to (95.9, 79.5), turned to 180 degrees
- moved REF** 0.87 mm to (170.2, 87.9)
- moved J1 0.40 mm to (111.7, 97.9)
- moved C3 0.39 mm to (100.6, 79.4)
- moved C2 0.37 mm to (119.6, 105.0)
- moved R2 0.05 mm to (130.5, 92.6)
- turned J2 to -90 degrees
Connections:
- HEEPidermis2 pad 15: /DSM_IN_GPIO_5 -> unconnected-(HEEPidermis2-Pad15)
- HEEPidermis2 pad 24: /VCO_N_VN0 -> unconnected-(HEEPidermis2-Pad24)
- HEEPidermis2 pad 28: /VCO_VN0_VDD -> unconnected-(HEEPidermis2-Pad28)
- HEEPidermis2 pad 29: /VCO_P_VN0 -> unconnected-(HEEPidermis2-Pad29)
- HEEPidermis2 pad 49: /GPIO_0 -> unconnected-(HEEPidermis2-Pad49)
- HEEPidermis2 pad 6: /EXIT_VALID -> unconnected-(HEEPidermis2-Pad6)
- HEEPidermis2 pad 7: /EXIT_VALUE -> unconnected-(HEEPidermis2-Pad7)
- HEEPidermis2 pad 9: /VCO_CNT_OVF -> unconnected-(HEEPidermis2-Pad9)
- J15 pad 15: /GND -> GND
- J15 pad 16: /GND -> GND
- J15 pad 27: /GND -> GND
- J15 pad 28: /GND -> GND
- J15 pad 5: /GND -> GND
- J15 pad 6: /GND -> GND
- J2 pad 24: /LC_DIR_GPIO_2 -> /LC_DIR_vs
- J2 pad 26: /LC_XING_GPIO_3 -> /LC_XING_vs
- J23 pad 2: /GPIO -> /GPIO_6
- J23 pad 4: /GPIO -> /GPIO.LED_R_1
- J23 pad 40: /GPIO -> /GPIO.LED_R_2
- J23 pad 42: /GPIO -> unconnected-(J23-Pin_42-Pad42)
- J23 pad 44: /GPIO -> unconnected-(J23-Pin_44-Pad44)
- J23 pad 46: /GPIO -> unconnected-(J23-Pin_46-Pad46)
- J23 pad 50: /GPIO -> unconnected-(J23-Pin_50-Pad50)
- J23 pad 52: /GPIO -> unconnected-(J23-Pin_52-Pad52)
- J23 pad 54: /GPIO -> unconnected-(J23-Pin_54-Pad54)
- J23 pad 56: /GPIO -> unconnected-(J23-Pin_56-Pad56)
- J23 pad 6: /GPIO -> /GPIO.LED_B_1
Routing:
- net /GPIO.LED_R_1: track 1.27 -> 46.2 mm, vias 0 -> 1
- net /GPIO_6: track 20.0 -> 64.5 mm, vias 0 -> 1
- net /GPIO.LED_B_1: track 1.27 -> 38.2 mm, vias 0 -> 1
- net /LC_DIR_GPIO_2: track 46.5 -> 16.6 mm, vias 1 -> 0
- net /LC_XING_GPIO_3: track 48.8 -> 21.7 mm, vias 1 -> 0
- net GND: track 214.2 -> 238.4 mm, vias 43 -> 472
- net /SUPPLY_IO_VDD: track 136.4 -> 113.7 mm, vias 15 -> 9
- net /LC_DIR_vs: track 0.00 -> 19.7 mm, vias 0 -> 1
- net /LC_XING_vs: track 0.00 -> 14.5 mm, vias 0 -> 1
- net /SPI_S_SCK: track 51.9 -> 65.6 mm
- net /SPI_S_MISO: track 51.4 -> 63.7 mm
- net /GPIO.LED_R_2: track 0.00 -> 10.2 mm
- net /SPI_S_MOSI: track 46.8 -> 56.6 mm
- net /SPI_S_CS: track 47.7 -> 54.7 mm
- net /CLOCK_vs: track 30.1 -> 34.3 mm
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- added copper zone on F.Cu, net /SUPPLY_IO_VDD
- added copper zone on In1.Cu, net /SUPPLY_IO_VDD
Other:
- board size 85.7 x 54 mm -> 85.7 x 58.6 mm
- board text added: "0"
- board text added: "1"
- board text added: "ACORE VDD"
- board text added: "AMUX VDD"
- board text added: "AMUX VOUT"
- board text added: "BOOT SEL"
- board text added: "CHANGE FOR CHRISTOPH'S CONNECTOR!"
- board text added: "CLOCK"
- board text added: "DCORE"
- board text added: "DCORE VDD"
- board text added: "FLASH EXEC"
- board text added: "GPIO 0"
- board text added: "IO VDD"
- board text added: "JTAG"
- board text added: "Juan Sapriza - 09/25 juan.sapriza@epfl.ch"
- board text added: "LDO REF"
- board text added: "LDO VBAT"
- board text added: "LDO VDD"
- board text added: "LDO VIN"
- board text added: "LDO VOUT"
- board text added: "LED"
- board text added: "MAINBOARD GPIO"
- board text added: "NVIN"
- board text added: "NVN0"
- board text added: "PVIN"
- board text added: "PVN0"
- board text added: "REF VDD"
- board text added: "RESET"
- board text added: "TDI TMS"
- board text added: "TDO TCK"
- board text added: "TESTPAD"
- board text added: "TO MAINBOARD"
- board text added: "TO VERSASENSE"
- board text added: "TP"
- board text added: "TRST nRST"
- board text added: "VALID"
- board text added: "VALUE"
- board text added: "VCO VDD"
- board text added: "VCO counter overflow"
- board text added: "VERSASENS GPIO"
- board text added: "VN0 VDD"
- board text added: "VREF VDD"
- board text added: "dLC Xing"
- board text added: "dLC dir"
- board text added: "iDAC1 IN"
- board text added: "iDAC1 OUT"
- board text added: "iDAC2 IN"
- board text added: "iDAC2 OUT"
- board text added: "iREF"
- board text added: "iREF VDD"
- board text added: "iREF1 out"
- board text added: "iREF2 out"
- board text added: "short to take clock clock from versasens"
- board text added: "short to take clock from SMA connector (or main board)"
- board text added: "short to take clock from main board"
- board text added: "vREF OUT"
- board text added: "x"
- board text added: "ΔΣ CLK"
- board text added: "ΔΣ IN"
- board text added: "↓RX TX↑"
- board text added: "◀"

Commit message: Uploaded gerbers
Parts:
- added J16: Conn_01x03, TestPoint:TestPoint_THTPad_1.0x1.0mm_Drill0.5mm, F.Cu at (105.3, 104.4)
- added J24: Conn_01x03, TestPoint:TestPoint_THTPad_1.0x1.0mm_Drill0.5mm, F.Cu at (109.5, 104.3)
- added J25: Conn_01x03, TestPoint:TestPoint_THTPad_1.0x1.0mm_Drill0.5mm, F.Cu at (96.2, 100.6)
- added J26: Conn_01x03, TestPoint:TestPoint_THTPad_1.0x1.0mm_Drill0.5mm, F.Cu at (97.2, 100.6)
- added J27: Conn_01x03, TestPoint:TestPoint_THTPad_1.0x1.0mm_Drill0.5mm, F.Cu at (94.0, 100.6)
- added J28: Conn_01x03, TestPoint:TestPoint_THTPad_1.0x1.0mm_Drill0.5mm, F.Cu at (95.1, 100.6)
- added J29: Conn_01x03, TestPoint:TestPoint_THTPad_1.0x1.0mm_Drill0.5mm, F.Cu at (149.6, 82.8)
- added J3: Conn_01x03, TestPoint:TestPoint_THTPad_1.0x1.0mm_Drill0.5mm, F.Cu at (108.1, 104.3)
- added J30: Conn_01x03, TestPoint:TestPoint_THTPad_1.0x1.0mm_Drill0.5mm, F.Cu at (165.3, 119.9)
- added J31: Conn_01x03, TestPoint:TestPoint_THTPad_1.0x1.0mm_Drill0.5mm, F.Cu at (97.4, 77.7)
- added J32: Conn_01x03, TestPoint:TestPoint_THTPad_1.0x1.0mm_Drill0.5mm, F.Cu at (99.0, 77.7)
- added J33: Conn_01x03, TestPoint:TestPoint_THTPad_1.0x1.0mm_Drill0.5mm, F.Cu at (102.8, 97.0)
- added J34: Conn_01x03, TestPoint:TestPoint_THTPad_1.0x1.0mm_Drill0.5mm, F.Cu at (102.5, 97.9)
- added J35: Conn_01x03, TestPoint:TestPoint_THTPad_1.0x1.0mm_Drill0.5mm, F.Cu at (102.2, 98.8)
- added J36: Conn_01x03, TestPoint:TestPoint_THTPad_1.0x1.0mm_Drill0.5mm, F.Cu at (102.8, 93.1)
- added J4: Conn_01x03, TestPoint:TestPoint_THTPad_1.0x1.0mm_Drill0.5mm, F.Cu at (106.7, 104.3)
- added R6: 0R, Resistor_SMD:R_0402_1005Metric, F.Cu at (176.1, 90.5)
- added R7: 0R, Resistor_SMD:R_0402_1005Metric, F.Cu at (176.0, 109.7)
- added REF**: leprechaun, heep_footprints:leprechaun, F.Cu at (106.3, 118.0)
- moved C2 1.30 mm to (118.3, 105.0)
Connections:
- J14 pad 1: /IDAC_2_IOUT -> Net-(J14-Pin_1)
- J18 pad 1: /IDAC_1_IOUT -> Net-(J18-Pin_1)
Routing:
- net /SPI_S_MISO: track 63.7 -> 74.9 mm
- net /SPI_S_MOSI: track 56.6 -> 67.3 mm
- net /SPI_S_CS: track 54.7 -> 60.4 mm
- net /SPI_S_SCK: track 65.6 -> 70.7 mm
- net /IDAC_2_IOUT: track 47.7 -> 44.9 mm
- net /IDAC_1_IOUT: track 40.8 -> 38.1 mm
- net Net-(J18-Pin_1): track 0.00 -> 1.68 mm
- net /SUPPLY_IO_VDD: track 113.7 -> 115.4 mm
- net Net-(J14-Pin_1): track 0.00 -> 1.58 mm
- net /LC_XING_vs: track 14.5 -> 14.8 mm, vias 1 -> 0
- net /LC_DIR_vs: vias 1 -> 0
- net GND: vias 472 -> 466
- net /nRST: vias 2 -> 1
Other:
- board size 85.7 x 58.6 mm -> 85.7 x 58.5 mm
- board text added: "CS"
- board text added: "Clock VS"
- board text added: "HEEPidermis is SoC for Bio-Z recording. It is based on the open-source platform X-HEEP. The digital back-end and behavioral models of the analog front-end are also open-source! Check the QR codes to see the repos :)"
- board text added: "MISO"
- board text added: "MOSI"
- board text added: "Populate to measure Short to inject"
- board text added: "SCK"
- board text added: "SPI flash"
- board text added: "SPIs"
- board text added: "Xing"
- board text added: "dLC"
- board text added: "dir"
- board text added: "nRST"
- board text added: "notes"
- board text added: "short to take clock from versasens"
- board text removed: "CHANGE FOR CHRISTOPH'S CONNECTOR!"
- board text removed: "dLC Xing"
- board text removed: "dLC dir"
- board text removed: "short to take clock clock from versasens"
