File: heepokranios-bo.kicad_sch (KiCad schematic)
At the start: 61 parts, among them J1 Conn_01x03, J10 Conn_Boaxial, J11 Conn_Boaxial, J12 Conn_01x03, J13 Conn_01x03, J14 Conn_01x03, J15 Conn_02x16_Odd_Even, J16 Conn_01x03, J17 Conn_02x10_Odd_Even, J18 Conn_01x03, J19 Conn_01x03, J2 5025983393, J20 Conn_01x03, J21 Conn_01x03, J22 Conn_01x03, J23 Conn_02x29_Top_Bottom, J24 Conn_01x03, J25 Conn_01x03, J26 Conn_01x03, J27 Conn_01x03, J28 Conn_01x03, J29 Conn_01x03, J3 Conn_01x03, J30 Conn_01x03, J31 Conn_01x03, J32 Conn_01x03, J33 Conn_01x03, J34 Conn_01x03, J35 Conn_01x03, J36 Conn_01x03, J37 Conn_01x02, J4 Conn_01x03, J5 Conn_01x03, J6 Conn_01x03, J7 Conn_01x03, J8 Conn_01x03, J9 Conn_Boaxial, SW1 SW_Push

Commit message: Added symbol and footprint of cheep boards connector
Parts:
- removed HEEPidermis2: 264-5205-01, Package_DFN_QFN:QFN-64-1EP_9x9mm_P0.5mm_EP3.4x3.4mm, symbol QFN64-scoket:264-5205-01
- added J38: ~, ESL-EPFL:cheep_board_connector, symbol cheep_board_connector:cheep_board_connector
Connections:
- net GPIO_6: now also J38.A1
- no-connect marks 63 -> 50
Other:
- note removed: "!! ADD A RESISTOR TO MEASURE current from iOUT"

Commit message: Initial draft of the schematic
Parts:
- removed J38: ~, ESL-EPFL:cheep_board_connector, symbol cheep_board_connector:cheep_board_connector
- added C12, C13, C14, C15, C16, C17, C18, C20, C22, C24, C26, C28, C30, C32, C35, C37, C39, C41, C43, C45: 100n, Capacitor_SMD:C_0603_1608Metric, symbol Device:C_Small
- added C19, C21, C23, C25, C27, C29, C31, C33, C34, C36, C38, C40, C42, C44, C46, C47, C48, C49, C50, C51: 1u, Capacitor_SMD:C_0603_1608Metric, symbol Device:C_Small
- added C52, C53, C54, C55, C56, C57, C58, C59, C60, C61, C62: 10u, Capacitor_SMD:C_0603_1608Metric, symbol Device:C_Small
- added D1: LED, symbol Device:LED
- added J100, J102, J104, J108, J110, J112, J113, J114, J117, J120, J123, J124, J125, J143, J144, J145, J146, J147, J148, J149, J150, J40, J41, J46, J47, J49, J53, J56, J58, J60, J62, J64, J66, J68, J70, J72, J74, J76, J78, J80, J82, J84, J88, J90, J92, J94, J96, J98: Conn_Boaxial, Connector_Coaxial:SMA_Amphenol_901-144_Vertical, symbol Connector:Conn_Coaxial
- added J101, J103, J107, J109, J111, J115, J116, J118, J119, J121, J122, J126, J127, J128, J129, J130, J131, J132, J133, J134, J135, J136, J137, J138, J139, J140, J141, J142, J42, J43, J44, J45, J57, J59, J61, J63, J65, J67, J69, J71, J73, J75, J77, J79, J81, J83, J85, J89, J91, J93, J95, J97, J99: Conn_01x03, Connector_PinHeader_1.27mm:PinHeader_1x01_P1.27mm_Vertical, symbol Connector_Generic:Conn_01x01
- added J105, J106, J50, J55: Conn_02x03_Odd_Even, symbol Connector_Generic:Conn_02x03_Odd_Even
- added J38: PGA_13x13, PGA_socket:PGA_13x13, symbol PGA_socket:PGA_13x13
- added J39: ~, ESL-EPFL:cheep_board_connector, symbol cheep_board_connector:cheep_board_connector
- added J48, J51, J52: Conn_02x02_Odd_Even, symbol Connector_Generic:Conn_02x02_Odd_Even
- added J54: Conn_02x04_Odd_Even, symbol Connector_Generic:Conn_02x04_Odd_Even
- added J86: ~, symbol heepokranios-bo-library:Conn_03x03
- added J87: Conn_01x05, symbol Connector_Generic:Conn_01x05
- added R10: 10k, symbol Device:R_US
- added R12: 1k, Resistor_SMD:R_0603_1608Metric, symbol Device:R
- added R13, R14: 1M, symbol Device:R_US
- added SW2: SW_Push, Button_Switch_SMD:SW_Push_1P1T_NO_CK_KMR2, symbol Switch:SW_Push
Connections:
- net GND: now also C12.2, C13.2, C14.2, C15.2, C16.2, C17.2, C18.2, C19.2, C20.2, C21.2, C22.2, C23.2, C24.2, C25.2, C26.2, C27.2, C28.2, C29.2, C30.2, C31.2, C32.2, C33.2, C34.2, C35.2, C36.2, C37.2, C38.2, C39.2, C40.2, C41.2, C42.2, C43.2, C44.2, C45.2, C46.2, C47.2, C48.2, C49.2, C50.2, C51.2, C52.1, C53.1, C54.1, C55.1, C56.1, C57.1, C58.1, C59.1, C60.1, C61.1, C62.1, J100.2 (Ext), J102.2 (Ext), J104.2 (Ext), J108.2 (Ext), J110.2 (Ext), J112.2 (Ext), J113.2 (Ext), J114.2 (Ext), J117.2 (Ext), J120.2 (Ext), J123.2 (Ext), J124.2 (Ext), J125.2 (Ext), J143.2 (Ext), J144.2 (Ext), J145.2 (Ext), J146.2 (Ext), J147.2 (Ext), J148.2 (Ext), J149.2 (Ext), J150.2 (Ext), J38.B1 (2), J38.B12 (76), J38.B5 (94), J38.B9 (82), J38.M12 (51), J38.M7 (37), J38.N1 (25), J38.N12 (48), J40.2 (Ext), J41.2 (Ext), J46.2 (Ext), J47.2 (Ext), J49.2 (Ext), J53.2 (Ext), J56.2 (Ext), J58.2 (Ext), J60.2 (Ext), J62.2 (Ext), J64.2 (Ext), J66.2 (Ext), J68.2 (Ext), J70.2 (Ext), J72.2 (Ext), J74.2 (Ext), J76.2 (Ext), J78.2 (Ext), J80.2 (Ext), J82.2 (Ext), J84.2 (Ext), J87.5 (Pin_5), J88.2 (Ext), J90.2 (Ext), J92.2 (Ext), J94.2 (Ext), J96.2 (Ext), J98.2 (Ext), R13.2, R14.2, SW2.2
- net nRST: now also J38.B2 (1), J39.B26, R12.1, SW2.1
- new net: J38.M3 (28), J56.1 (In), J57.1 (Pin_1)
- new net: J38.N2 (27), J60.1 (In), J61.1 (Pin_1)
- new net: J38.J12 (57), J90.1 (In), J91.1 (Pin_1)
- new net: J117.1 (In), J38.D2 (5), J45.1 (Pin_1), J47.1 (In)
- new net: J38.L8 (42), J74.1 (In), J75.1 (Pin_1)
- new net: J38.K13 (56), J88.1 (In), J89.1 (Pin_1)
- new net: D1.1 (K), J38.A1 (100)
- new net: D1.2 (A), R10.2
- new net: J51.3 (Pin_3), J52.2 (Pin_2)
- new net: J38.J13 (58), J92.1 (In), J93.1 (Pin_1)
- new net: J38.H11 (59), J94.1 (In), J95.1 (Pin_1)
- new net: J124.1 (In), J38.C1 (4), J44.1 (Pin_1)
- new net: J38.N11 (47), J80.1 (In), J81.1 (Pin_1)
- new net: J38.F1 (11), J41.1 (In), J43.1 (Pin_1)
- new net: J38.H12 (60), J96.1 (In), J97.1 (Pin_1)
- new net: J38.E1 (8), J40.1 (In), J42.1 (Pin_1)
- new net: J38.N7 (39), J84.1 (In), J85.1 (Pin_1)
- new net: J38.H13 (61), J98.1 (In), J99.1 (Pin_1)
- new net: J38.N8 (40), J70.1 (In), J71.1 (Pin_1)
- new net: J38.M8 (41), J72.1 (In), J73.1 (Pin_1)
- new net: J100.1 (In), J101.1 (Pin_1), J38.F13 (65)
- new net: J38.N13 (50), J82.1 (In), J83.1 (Pin_1)
- new net: J102.1 (In), J103.1 (Pin_1), J38.F12 (66)
- new net: J38.M4 (30), J62.1 (In), J63.1 (Pin_1)
- new net: J38.M5 (32), J66.1 (In), J67.1 (Pin_1)
- new net: J38.N10 (45), J78.1 (In), J79.1 (Pin_1)
- new net: J38.N3 (29), J58.1 (In), J59.1 (Pin_1)
- new net: J38.N4 (31), J64.1 (In), J65.1 (Pin_1)
- new net: J38.N6 (36), J68.1 (In), J69.1 (Pin_1)
- new net: J38.N9 (43), J76.1 (In), J77.1 (Pin_1)
- new net: J52.4 (Pin_4), J53.1 (In), R14.1
- new net CG_BPE_VDD: C38.1, C39.1, C54.2, J38.G12 (62), J39.B41
- new net CG_CH_01_ADCS_VDD: C55.2, J39.B40, J86.1, J86.2, J86.3
- new net CG_CH_01_LNA_VDD: C53.2, J106.1 (Pin_1), J106.2 (Pin_2), J39.B45
- new net CG_DATA_CLK_VIN: C58.2, J39.B16, J48.3 (Pin_3)
- new net CG_IIN: J39.B11, J51.1 (Pin_1)
- new net CG_LC_VDD: C30.1, C31.1, C61.2, J38.L2 (24), J39.B6
- new net CG_LNA_VCM: C52.2, J39.B46, J50.1 (Pin_1), J50.2 (Pin_2)
- new net CG_RECT_VOUT: C59.2, J105.1 (Pin_1), J105.2 (Pin_2), J39.B15
- new net CG_REFS_VDD: C62.2, J39.B5, J55.1 (Pin_1), J55.2 (Pin_2)
- new net CG_VDD: C16.1, C17.1, C50.1, C51.1, C57.2, J38.19 (83), J38.A5 (93), J39.B35
- new net CG_VDD_IO: C12.1, C13.1, C14.1, C15.1, C46.1, C47.1, C48.1, C49.1, C56.2, J38.A12 (77), J38.C2 (3), J38.M13 (52), J38.M2 (26), J39.B36
- new net CG_VREF: C60.2, J39.B10, J54.3 (Pin_3), J54.5 (Pin_5)
- new net CH_0_DSM_VDD: C34.1, C35.1, J38.G13 (64), J86.4
- new net CH_0_LNA_VDD: C44.1, C45.1, J106.3 (Pin_3), J38.L12 (53)
- new net CH_0_PD_VCO_VDD: C36.1, C37.1, J38.G11 (63), J86.5
- new net CH_1_DSM_VDD: C40.1, C41.1, J38.K12 (55), J86.6
- new net CH_1_VDD: C42.1, C43.1, J106.4 (Pin_4), J38.L13 (54)
- new net CH_234_VDD: C28.1, C29.1, J38.M1 (23), J55.3 (Pin_3)
- new net CLK_32k: J39.C32
- new net DMUX_0: J127.1 (Pin_1), J128.1 (Pin_1), J143.1 (In), J38.A13 (75)
- new net DMUX_1: J129.1 (Pin_1), J130.1 (Pin_1), J144.1 (In), J38.C12 (74)
- new net DMUX_2: J131.1 (Pin_1), J132.1 (Pin_1), J145.1 (In), J38.B13 (73)
- new net DMUX_3: J133.1 (Pin_1), J134.1 (Pin_1), J146.1 (In), J38.C13 (72)
- new net DMUX_4: J135.1 (Pin_1), J136.1 (Pin_1), J147.1 (In), J38.D12 (71)
- new net DMUX_5: J137.1 (Pin_1), J138.1 (Pin_1), J148.1 (In), J38.D13 (70)
- new net DMUX_6: J139.1 (Pin_1), J140.1 (Pin_1), J149.1 (In), J38.E12 (69)
- new net DMUX_7: J141.1 (Pin_1), J142.1 (Pin_1), J150.1 (In), J38.E13 (68)
- new net IMIRROR_IIN: J38.K1 (20), J51.2 (Pin_2), J51.4 (Pin_4)
- new net IMIRROR_IOUT: J38.F3 (9), J49.1 (In), R13.1
- new net IREF_IOUT: J38.J2 (19), J52.1 (Pin_1), J52.3 (Pin_3)
- new net JTAG_TCK: J38.A2 (98), J39.B24
- new net JTAG_TDI: J38.A3 (97), J39.C25
- new net JTAG_TDO: J38.B3 (99), J39.C24
- new net JTAG_TMS: J38.B4 (96), J39.B25
- new net JTAG_TRST: J38.A4 (95), J39.C26
- new net LNA_VCM_VIN: C32.1, C33.1, J38.M6 (35), J50.3 (Pin_3)
- new net PLL_CLK: J114.1 (In), J39.C29
- new net REFS_VDD: C24.1, C25.1, J38.J1 (18), J55.4 (Pin_4)
- new net UART_CHEEP_RX: J38.A10 (81), J39.C22
- new net UART_CHEEP_TX: J38.B10 (80), J39.B22
- new net VDD_IO: J39.C31, R10.1, R12.2
- new net VREF_0V4_BUFF: J38.L6 (34), J50.5 (Pin_5), J50.6 (Pin_6)
- new net VREF_0V5_BUFF: J38.K2 (21), J54.7 (Pin_7)
- new net VREF_0V5_UNBUFF: J38.H1 (15), J54.1 (Pin_1)
- new net VREF_0V6_BUFF: J38.E2 (7), J48.1 (Pin_1)
- new net VREF_EN: J105.4 (Pin_4), J38.G3 (13)
- new net VREF_HVDD: C20.1, C21.1, J105.3 (Pin_3), J38.G1 (14)
- new net VREF_VIN: C26.1, C27.1, J38.L1 (22), J54.6 (Pin_6), J54.8 (Pin_8)
- new net VSS: J39.B13, J39.B18, J39.B23, J39.B28, J39.B29, J39.B32, J39.B33, J39.B38, J39.B43, J39.B8, J39.C13, J39.C18, J39.C23, J39.C28, J39.C30, J39.C33, J39.C38, J39.C43, J39.C8
- new net WPDT_BLOCKS_VIN: J38.N5 (33), J50.4 (Pin_4)
- new net WPDT_DATA_CLK_VIN: C18.1, C19.1, J38.D1 (6), J48.2 (Pin_2), J48.4 (Pin_4)
- new net WPDT_LDO_VIN: C22.1, C23.1, J38.H2 (16), J54.2 (Pin_2), J54.4 (Pin_4)
- new net WPDT_LDO_VOUT: J106.5 (Pin_5), J106.6 (Pin_6), J38.H3 (17), J55.5 (Pin_5), J55.6 (Pin_6), J86.7, J86.8, J86.9
- new net WPDT_RECT_VOUT: J105.5 (Pin_5), J105.6 (Pin_6), J38.G2 (12)
- new net WPDT_SCKI: J108.1 (In), J109.1 (Pin_1), J119.1 (Pin_1), J38.B6 (91)
- new net WPDT_SCKO: J110.1 (In), J111.1 (Pin_1), J38.A6 (90)
- new net WPDT_SDI: J104.1 (In), J107.1 (Pin_1), J118.1 (Pin_1), J38.C6 (92)
- new net reg2ser_scki: J125.1 (In), J126.1 (Pin_1)
- new net spi_slave_cs: J38.C8 (84), J87.4 (Pin_4)
- new net spi_slave_miso: J38.B8 (85), J87.3 (Pin_3)
- new net spi_slave_mosi: J122.1 (Pin_1), J123.1 (In), J38.B7 (87), J87.1 (Pin_1)
- new net spi_slave_sck: J113.1 (In), J116.1 (Pin_1), J38.A8 (86), J87.2 (Pin_2)
- new net wpdt2ser_scko: J112.1 (In), J115.1 (Pin_1), J38.A7 (89)
- new net wpdt2ser_sdo: J120.1 (In), J121.1 (Pin_1), J38.C7 (88)
- no-connect marks 50 -> 163
Other:
- note added: "(!) Choose low Vt diode"
- note added: "(!) Connect via the matrix!"
- note added: "(!) Watch out, these pins are also available in the SPI connector"
- note added: "< debug only"
- note added: "< reg2ser_scki (dmux 5)"
- note added: "< reg2ser_scko (dmux 3)"
- note added: "< reg2ser_sdo (dmux 2)"
- note added: "Antenna connector"
- note added: "BPE VIN"
- note added: "BPE VOUT"
- note added: "Ch 0"
- note added: "Ch 1"
- note added: "Ch 2"
- note added: "Ch 3"
- note added: "Ch 4"
- note added: "Choose ref clk"
- note added: "Clock selection"
- note added: "Connect the inputs to the chewing gum"
- note added: "Connect the inputs to the chip's outputs"
- note added: "Current monitoring"
- note added: "DSM VIN"
- note added: "Decoupling next to each input to the board"
- note added: "Decoupling next to each input to the chip"
- note added: "Decoupling on the chip's power"
- note added: "Digital multiplexed bits"
- note added: "LNA"
- note added: "Options for the voltage reference"
- note added: "PLL CLK > REF CLK > WPDT REF CLK > SIGNAL GEN >"
- note added: "Reference for High (dirty) voltage"
- note added: "Reference for the channel's ADCs"
- note added: "Reference for the channel's LNAs"
- note added: "Reference for the data clock's VCO"
- note added: "SPI slave connector"
- note added: "SoC reset (active low)"
- note added: "Use clocks for sth else"
- note added: "VCM/WPDT blocks"
- note added: "VCO VIN"
- note added: "VDD for standard analog blocks"
- note added: "WPDT communication"
- moved on the sheet: C1, C10, C11, C2, C3, C4, C5, C6, C7, C8, C9, HEEPidermis1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

Commit message: Initial floorplannig
Parts:
- removed C1, C10, C2, C3, C4, C5, C6, C7, C8, C9: 100n, Capacitor_SMD:C_0603_1608Metric, symbol Device:C_Small
- removed C11: Cp_skin, Capacitor_SMD:C_0603_1608Metric, symbol Device:C_Small
- removed HEEPidermis1: 264-5205-01, CONN_5205_3MM, symbol QFN64-scoket:264-5205-01
- removed J1, J101, J103, J107, J109, J111, J115, J116, J118, J119, J121, J122, J126, J127, J128, J129, J130, J131, J132, J133, J134, J135, J136, J137, J138, J139, J14, J140, J141, J142, J18, J42, J43, J44, J45, J57, J59, J61, J63, J65, J67, J69, J71, J73, J75, J77, J79, J81, J83, J85, J89, J91, J93, J95, J97, J99: Conn_01x03, Connector_PinHeader_1.27mm:PinHeader_1x01_P1.27mm_Vertical, symbol Connector_Generic:Conn_01x01
- removed J10, J100, J102, J104, J108, J11, J110, J112, J113, J114, J117, J120, J123, J124, J125, J143, J144, J145, J146, J147, J148, J149, J150, J40, J41, J46, J47, J49, J53, J56, J58, J60, J62, J64, J66, J68, J70, J72, J74, J76, J78, J80, J82, J84, J88, J9, J90, J92, J94, J96, J98: Conn_Boaxial, Connector_Coaxial:SMA_Amphenol_901-144_Vertical, symbol Connector:Conn_Coaxial
- removed J12, J13, J19, J20, J7: Conn_01x03, Connector_PinHeader_2.54mm:PinHeader_1x03_P2.54mm_Vertical, symbol Connector_Generic:Conn_01x03
- removed J15: Conn_02x16_Odd_Even, Connector_PinHeader_2.54mm:PinHeader_02x16_P2.54mm_Vertical, symbol Connector_Generic:Conn_02x16_Odd_Even
- removed J16, J24, J25, J26, J27, J28, J29, J3, J30, J31, J32, J33, J34, J35, J36, J4: Conn_01x03, TestPoint_THTPad_1.0x1.0mm_Drill0.5mm, symbol Connector_Generic:Conn_01x01
- removed J17: Conn_02x10_Odd_Even, Connector_PinHeader_2.54mm:PinHeader_2x10_P2.54mm_Vertical, symbol Connector_Generic:Conn_02x10_Odd_Even
- removed J2: 5025983393, heep_footprints:CONN_502598-3393_MOL, symbol 2025-09-27_11-33-13:5025983393
- removed J23: Conn_02x29_Top_Bottom, Connector_PinHeader_2.54mm:PinHeader_2x32_P2.54mm_Vertical, symbol Connector_Generic:Conn_02x32_Odd_Even
- removed J37: Conn_01x02, Connector_PinHeader_1.27mm:PinHeader_1x04_P1.27mm_Vertical, symbol Connector_Generic:Conn_01x04
- removed J5, J6: Conn_01x03, Connector_PinHeader_1.27mm:PinHeader_2x03_P1.27mm_Vertical, symbol Connector_Generic:Conn_02x03_Odd_Even
- removed J51, J52: Conn_02x02_Odd_Even, symbol Connector_Generic:Conn_02x02_Odd_Even
- removed J8: Conn_01x03, Connector_PinHeader_1.27mm:PinHeader_2x02_P1.27mm_Vertical, symbol Connector_Generic:Conn_02x02_Odd_Even
- removed R1, R2, R3: 0R, X-MODs_PcbLib:R0402, symbol Device:R
- removed R13, R14: 1M, symbol Device:R_US
- removed R4: 1k, Resistor_SMD:R_0603_1608Metric, symbol Device:R
- removed R5: 10k, Resistor_SMD:R_0603_1608Metric, symbol Device:R
- removed R6, R7: 0R, Resistor_SMD:R_0402_1005Metric, symbol Device:R
- removed R8: Rs_skin, Resistor_SMD:R_0603_1608Metric, symbol Device:R
- removed R9: Rp_skin, Resistor_SMD:R_0603_1608Metric, symbol Device:R
- removed SW1: SW_Push, Button_Switch_SMD:SW_Push_1P1T_NO_CK_KMR2, symbol Switch:SW_Push
- removed U1: ~, heep_footprints:SPDT-2pos-CAS-D20B1, symbol Switch:SW_DPDT_x2
- added J1, J9: Conn_02x02_Odd_Even, Connector_PinHeader_2.54mm:PinHeader_2x02_P2.54mm_Vertical, symbol Connector_Generic:Conn_02x02_Odd_Even
- added J12: Conn_01x08_Pin, Connector_PinHeader_2.54mm:PinHeader_1x08_P2.54mm_Vertical, symbol Connector:Conn_01x08_Pin
- added J13: Conn_01x08_Socket, Connector_PinHeader_2.54mm:PinHeader_1x08_P2.54mm_Vertical, symbol Connector:Conn_01x08_Socket
- added R1, R2: 1M, Resistor_SMD:R_0603_1608Metric, symbol Device:R_US
- added S1, S10, S11, S12, S13, S14, S15, S16, S17, S18, S19, S2, S20, S21, S22, S23, S24, S25, S26, S27, S28, S29, S3, S30, S31, S32, S33, S34, S35, S36, S37, S38, S39, S4, S40, S41, S42, S43, S44, S45, S46, S47, S48, S49, S5, S6, S7, S8, S9: SMA connector, heepokranios-bo-library:SMA_w_tp, symbol heepokranios-bo-library:SMA_w_tp
- D1: footprint (none) -> LED_SMD:LED_0603_1608Metric
- J2: renamed from J48; footprint (none) -> Connector_PinHeader_2.54mm:PinHeader_2x02_P2.54mm_Vertical
- J20: renamed from J87; footprint (none) -> Connector_PinHeader_2.54mm:PinHeader_1x05_P2.54mm_Vertical
- J21, J22: footprint Connector_PinHeader_1.27mm:PinHeader_1x01_P1.27mm_Vertical -> Connector_PinHeader_2.54mm:PinHeader_1x01_P2.54mm_Vertical
- J3: renamed from J55; footprint (none) -> Connector_PinHeader_2.54mm:PinHeader_2x03_P2.54mm_Vertical
- J4: renamed from J50; footprint (none) -> Connector_PinHeader_2.54mm:PinHeader_2x03_P2.54mm_Vertical
- J5: renamed from J105; footprint (none) -> Connector_PinHeader_2.54mm:PinHeader_2x03_P2.54mm_Vertical
- J6: renamed from J54; footprint (none) -> Connector_PinHeader_2.54mm:PinHeader_2x04_P2.54mm_Vertical
- J7: renamed from J86; footprint (none) -> heepokranios-bo-library:Conn_3x03
- J8: renamed from J106; footprint (none) -> Connector_PinHeader_2.54mm:PinHeader_2x03_P2.54mm_Vertical
- R4: renamed from R10; footprint (none) -> Resistor_SMD:R_0603_1608Metric
- renumbered C12 to C1, C28 to C10, C30 to C11, C46 to C12, C19 to C13, C21 to C14, C23 to C15, C25 to C16, C27 to C17, C29 to C18, C31 to C19, C13 to C2, C52 to C20, C53 to C21, C54 to C22, C55 to C23, C56 to C24, C57 to C25, C47 to C26, C48 to C27, C49 to C28, C58 to C29, C14 to C3, C59 to C30, C60 to C31, C61 to C32, C62 to C33, C33 to C34, C34 to C35, C38 to C37, C40 to C38, C42 to C39, C15 to C4, C44 to C40, C16 to C41, C32 to C42, C35 to C43, C37 to C44, C39 to C45, C41 to C46, C43 to C47, C45 to C48, C17 to C49, C18 to C5, C20 to C6, C22 to C7, C24 to C8, C26 to C9, J39 to J10, J38 to J11, R12 to R3, SW2 to SW1
Connections:
- net VCO_N_VIN is gone; now on net WPDT_SCKI: J21.1 (Pin_1)
- net VCO_P_VIN is gone; now on net WPDT_SDI: J22.1 (Pin_1)
- net CG_IIN: now also J9.1 (Pin_1)
- net DMUX_0: now also J12.1 (Pin_1), J13.1 (Pin_1), S21.1
- net DMUX_1: now also J12.2 (Pin_2), J13.2 (Pin_2), S22.1
- net DMUX_2: now also J12.3 (Pin_3), J13.3 (Pin_3), S23.1
- net DMUX_3: now also J12.4 (Pin_4), J13.4 (Pin_4), S24.1
- net DMUX_4: now also J12.5 (Pin_5), J13.5 (Pin_5), S25.1
- net DMUX_5: now also J12.6 (Pin_6), J13.6 (Pin_6), S26.1
- net DMUX_6: now also J12.7 (Pin_7), J13.7 (Pin_7), S27.1
- net DMUX_7: now also J12.8 (Pin_8), J13.8 (Pin_8), S28.1
- net GND: now also R1.2, R2.2, S1.2, S10.2, S11.2, S12.2, S13.2, S14.2, S15.2, S16.2, S17.2, S18.2, S19.2, S2.2, S20.2, S21.2, S22.2, S23.2, S24.2, S25.2, S26.2, S27.2, S28.2, S29.2, S3.2, S30.2, S31.2, S32.2, S33.2, S34.2, S35.2, S36.2, S37.2, S38.2, S39.2, S4.2, S40.2, S41.2, S42.2, S43.2, S44.2, S45.2, S46.2, S47.2, S48.2, S49.2, S5.2, S6.2, S7.2, S8.2, S9.2
- net IMIRROR_IIN: now also J9.2 (Pin_2), J9.4 (Pin_4)
- net IMIRROR_IOUT: now also R2.1, S2.1
- net IREF_IOUT: now also J1.1 (Pin_1), J1.3 (Pin_3)
- net PLL_CLK: now also S7.1
- net WPDT_SCKI: now also S42.1
- net WPDT_SCKO: now also S43.1
- net WPDT_SDI: now also S41.1
- net reg2ser_scki: now also S46.1
- net spi_slave_mosi: now also S48.1
- net spi_slave_sck: now also S47.1
- net wpdt2ser_scko: now also S44.1
- net wpdt2ser_sdo: now also S45.1
- net at J11.M3 (28): now also S11.1
- net at J11.N2 (27): now also S10.1
- net at J11.J12 (57): now also S35.1
- net at J11.D2 (5): now also S6.1, S9.1
- net at J11.L8 (42): now also S20.1
- net at J11.K13 (56): now also S36.1
- net at J11.J13 (58): now also S34.1
- net at J11.H11 (59): now also S33.1
- net at J11.C1 (4): now also S5.1, S8.1
- net at J11.N11 (47): now also S38.1
- net at J11.F1 (11): now also S4.1
- net at J11.H12 (60): now also S32.1
- net at J11.E1 (8): now also S3.1
- net at J11.N7 (39): now also S17.1
- net at J11.H13 (61): now also S31.1
- net at J11.N8 (40): now also S18.1
- net at J11.M8 (41): now also S19.1
- net at J11.F13 (65): now also S30.1
- net at J11.N13 (50): now also S37.1
- net at J11.F12 (66): now also S29.1
- net at J11.M4 (30): now also S13.1
- net at J11.M5 (32): now also S15.1
- net at J11.N10 (45): now also S39.1
- net at J11.N3 (29): now also S12.1
- net at J11.N4 (31): now also S14.1
- net at J11.N6 (36): now also S16.1
- net at J11.N9 (43): now also S40.1, S49.1
- net at J10.A1: now also J10.A2
- new net: J1.4 (Pin_4), R1.1, S1.1
- new net: J1.2 (Pin_2), J9.3 (Pin_3)
- no-connect marks 163 -> 113
Other:
- note added: "(!) Make one of these columsn FEMALE"
- note removed: "SUPPLY_DCORE_VDD was not connected on the chip"
- moved on the sheet: J2, J3, J4, J5, J6, J7, J8, R3, SW1
