File: heepokranios-bo.kicad_pcb (KiCad board)
At the start: 4 copper layers, 142.2 x 15.4 mm, 122 parts, among them J1 Conn_02x02_Odd_Even, J11 PGA_13x13, J12 Conn_01x08_Pin, J13 Conn_01x08_Socket, J2 Conn_02x02_Odd_Even, J20 Conn_01x05, J21 Conn_01x03, J22 Conn_01x03, J3 Conn_02x03_Odd_Even, J4 Conn_02x03_Odd_Even, J5 Conn_02x03_Odd_Even, J6 Conn_02x04_Odd_Even, J8 Conn_02x03_Odd_Even, J9 Conn_02x02_Odd_Even, SW1 SW_Push

Commit message: In the process of floorplanning the pcb
Parts:
- moved J3 227.8 mm to (40.6, 137.2)
- moved J4 226.1 mm to (50.8, 137.2)
- moved J5 224.3 mm to (61.0, 137.2)
- moved J8 222.6 mm to (71.1, 137.2)
- moved J1 213.1 mm to (53.3, 121.9)
- moved J9 197.1 mm to (53.3, 111.8)
- moved J6 195.2 mm to (68.6, 104.1)
- moved J2 172.5 mm to (68.6, 83.8), turned to 90 degrees
- moved J7 136.8 mm to (132.6, 93.2)
Changed lines of the file:
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@@
 	(footprint "Connector_PinHeader_2.54mm:PinHeader_2x03_P2.54mm_Vertical"
 		(layer "F.Cu")
-		(at 179.2576 -43.67)
+		(at 40.64 137.16)
 		(descr "Through hole straight pin header, 2x03, 2.54mm pitch, double rows")
 		(tags "Through hole pin header THT 2x03 2.54mm double row")
@@
 	(footprint "Connector_PinHeader_2.54mm:PinHeader_2x03_P2.54mm_Vertical"
 		(layer "F.Cu")
-		(at 200.8576 -43.67)
+		(at 71.12 137.16)
 		(descr "Through hole straight pin header, 2x03, 2.54mm pitch, double rows")
 		(tags "Through hole pin header THT 2x03 2.54mm double row")
@@
 	(footprint "Connector_PinHeader_2.54mm:PinHeader_2x03_P2.54mm_Vertical"
 		(layer "F.Cu")
-		(at 193.6576 -43.67)
+		(at 60.96 137.16)
 		(descr "Through hole straight pin header, 2x03, 2.54mm pitch, double rows")
 		(tags "Through hole pin header THT 2x03 2.54mm double row")
@@
 	(footprint "Connector_PinHeader_2.54mm:PinHeader_2x02_P2.54mm_Vertical"
 		(layer "F.Cu")
-		(at 208.6076 -16.84)
+		(at 68.58 83.82 90)
 		(descr "Through hole straight pin header, 2x02, 2.54mm pitch, double rows")
 		(tags "Through hole pin header THT 2x02 2.54mm double row")
 		(property "Reference" "J2"
-			(at 1.27 -2.33 0)
+			(at 5.08 2.54 180)
 			(layer "F.SilkS")
 			(effects
@@
 		)
 		(property "Value" "Conn_02x02_Odd_Even"
-			(at 1.27 4.87 0)
+			(at 1.27 4.87 90)
 			(layer "F.Fab")
 			(effects
@@
 		)
 		(property "Datasheet" "~"
-			(at 0 0 0)
+			(at 0 0 90)
 			(unlocked yes)
 			(layer "F.Fab")
@@
 		)
 		(property "Description" "Generic connector, double row, 02x02, odd/even pin numbering scheme (row 1 odd numbers, row 2 even numbers), script generated (kicad-library-utils/schlib/autogen/connector/)"
-			(at 0 0 0)
+			(at 0 0 90)
 			(unlocked yes)
 			(layer "F.Fab")
@@
 		(attr through_hole)
 		(fp_line
-			(start -1.33 -1.33)
-			(end 0 -1.33)
+			(start 3.87 -1.33)
+			(end 3.87 3.87)
 			(stroke
 				(width 0.12)
@@
 		)
 		(fp_line
-			(start -1.33 0)
-			(end -1.33 -1.33)
+			(start 1.27 -1.33)
+			(end 3.87 -1.33)
 			(stroke
 				(width 0.12)
@@
 		)
 		(fp_line
-			(start -1.33 1.27)
-			(end -1.33 3.87)
+			(start -1.33 -1.33)
+			(end 0 -1.33)
 			(stroke
 				(width 0.12)
@@
 		)
 		(fp_line
-			(start -1.33 1.27)
-			(end 1.27 1.27)
+			(start -1.33 0)
+			(end -1.33 -1.33)
 			(stroke
 				(width 0.12)
@@
 		)
 		(fp_line
-			(start -1.33 3.87)
-			(end 3.87 3.87)
+			(start 1.27 1.27)
+			(end 1.27 -1.33)
 			(stroke
 				(width 0.12)
@@
 		)
 		(fp_line
-			(start 1.27 -1.33)
-			(end 3.87 -1.33)
+			(start -1.33 1.27)
+			(end 1.27 1.27)
 			(stroke
 				(width 0.12)
@@
 		)
 		(fp_line
-			(start 1.27 1.27)
-			(end 1.27 -1.33)
+			(start -1.33 1.27)
+			(end -1.33 3.87)
 			(stroke
 				(width 0.12)
@@
 		)
 		(fp_line
-			(start 3.87 -1.33)
+			(start -1.33 3.87)
 			(end 3.87 3.87)
 			(stroke
@@
 		)
 		(fp_line
-			(start -1.8 -1.8)
-			(end -1.8 4.35)
+			(start 4.35 -1.8)
+			(end -1.8 -1.8)
 			(stroke
 				(width 0.05)
@@
 		)
 		(fp_line
-			(start -1.8 4.35)
-			(end 4.35 4.35)
+			(start -1.8 -1.8)
+			(end -1.8 4.35)
 			(stroke
 				(width 0.05)
@@
 		)
 		(fp_line
-			(start 4.35 -1.8)
-			(end -1.8 -1.8)
+			(start 4.35 4.35)
+			(end 4.35 -1.8)
 			(stroke
 				(width 0.05)
@@
 		)
 		(fp_line
-			(start 4.35 4.35)
-			(end 4.35 -1.8)
+			(start -1.8 4.35)
+			(end 4.35 4.35)
 			(stroke
 				(width 0.05)
@@
 		)
 		(fp_line
-			(start -1.27 0)
-			(end 0 -1.27)
+			(start 3.81 -1.27)
+			(end 3.81 3.81)
 			(stroke
 				(width 0.1)
@@
 		)
 		(fp_line
-			(start -1.27 3.81)
-			(end -1.27 0)
+			(start 0 -1.27)
+			(end 3.81 -1.27)
 			(stroke
 				(width 0.1)
@@
 		)
 		(fp_line
-			(start 0 -1.27)
-			(end 3.81 -1.27)
+			(start -1.27 0)
+			(end 0 -1.27)
 			(stroke
 				(width 0.1)
@@
 		)
 		(fp_line
-			(start 3.81 -1.27)
-			(end 3.81 3.81)
+			(start 3.81 3.81)
+			(end -1.27 3.81)
 			(stroke
 				(width 0.1)
@@
 		)
 		(fp_line
-			(start 3.81 3.81)
-			(end -1.27 3.81)
+			(start -1.27 3.81)
+			(end -1.27 0)
 			(stroke
 				(width 0.1)
@@
 		)
 		(fp_text user "${REFERENCE}"
-			(at 1.27 1.27 90)
+			(at 1.27 1.27 0)
 			(layer "F.Fab")
 			(effects
@@
 		)
 		(pad "1" thru_hole rect
-			(at 0 0)
+			(at 0 0 90)
 			(size 1.7 1.7)
 			(drill 1)
@@
 		)
 		(pad "2" thru_hole oval
-			(at 2.54 0)
+			(at 2.54 0 90)
 			(size 1.7 1.7)
 			(drill 1)
@@
 		)
 		(pad "3" thru_hole oval
-			(at 0 2.54)
+			(at 0 2.54 90)
 			(size 1.7 1.7)
 			(drill 1)
@@
 		)
 		(pad "4" thru_hole oval
-			(at 2.54 2.54)
+			(at 2.54 2.54 90)
 			(size 1.7 1.7)
 			(drill 1)
@@
 	(footprint "heepokranios-bo-library:Conn_3x03"
 		(layer "F.Cu")
-		(at 197.7326 -27.112)
+		(at 132.5626 93.218)
 		(property "Reference" "J7"
-			(at -0.1524 0.5588 0)
+			(at 4.5974 -9.398 0)
 			(unlocked yes)
 			(layer "F.SilkS")
@@
 	(footprint "Connector_PinHeader_2.54mm:PinHeader_2x03_P2.54mm_Vertical"
 		(layer "F.Cu")
-		(at 186.4576 -43.67)
+		(at 50.8 137.16)
 		(descr "Through hole straight pin header, 2x03, 2.54mm pitch, double rows")
 		(tags "Through hole pin header THT 2x03 2.54mm double row")
@@
 	(footprint "Connector_PinHeader_2.54mm:PinHeader_2x02_P2.54mm_Vertical"
 		(layer "F.Cu")
-		(at 208.6076 -9.64)
+		(at 53.34 111.76)
 		(descr "Through hole straight pin header, 2x02, 2.54mm pitch, double rows")
 		(tags "Through hole pin header THT 2x02 2.54mm double row")
@@
 	(footprint "Connector_PinHeader_2.54mm:PinHeader_2x04_P2.54mm_Vertical"
 		(layer "F.Cu")
-		(at 215.8076 -24.04)
+		(at 68.58 104.14)
 		(descr "Through hole straight pin header, 2x04, 2.54mm pitch, double rows")
 		(tags "Through hole pin header THT 2x04 2.54mm double row")
@@
 	(footprint "Connector_PinHeader_2.54mm:PinHeader_2x02_P2.54mm_Vertical"
 		(layer "F.Cu")
-		(at 208.6076 -24.04)
+		(at 53.34 121.92)
 		(descr "Through hole straight pin header, 2x02, 2.54mm pitch, double rows")
 		(tags "Through hole pin header THT 2x02 2.54mm double row")

Commit message: Initial floorplanning
Parts:
- moved SW1 163.3 mm to (75.7, 70.3)
- moved J21 110.5 mm to (119.4, 61.0)
- moved J22 103.6 mm to (124.5, 61.0)
- moved J12 85.1 mm to (127.0, 43.2), turned to -90 degrees
- moved J13 68.3 mm to (127.0, 53.0), turned to -90 degrees
- moved J20 38.4 mm to (154.9, 43.2), turned to -90 degrees
- moved S25 32.3 mm to (139.7, 49.1), turned to 180 degrees
- moved S28 29.7 mm to (170.2, 49.1), turned to 180 degrees
- moved S24 27.8 mm to (139.7, 75.5), turned to 0 degrees
- moved S21 24.9 mm to (170.2, 75.5), turned to 0 degrees
- moved S26 24.0 mm to (149.9, 49.1), turned to 180 degrees
- moved S41 23.5 mm to (127.0, 75.5)
- moved S42 23.5 mm to (116.8, 75.5)
- moved S43 23.5 mm to (104.1, 75.5)
- moved S27 22.9 mm to (160.0, 49.1), turned to 180 degrees
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Other:
- board size 142.2 x 15.4 mm -> 119.6 x 15.7 mm
