File: gpio-playground/gpio-playground.kicad_sch (KiCad schematic)
At the start: 42 parts, among them J1 Conn_02x03_Odd_Even, J2 Conn_02x08_Odd_Even, SW1 SW_Push, SW2 SW_Push, SW3 SW_Push, SW4 SW_Push, SW5 SW_Push, SW6 SW_Push, SW7 SW_Push, SW8 SW_Push, U1 BIWIN_DTS04GE_SMD, U2 BIWIN_DTS04GE_SMD, U3 74AHC244

Commit message: Added gpio playground PCB
Connections:
- net DMUX_4: now also U2.4, U3.2 (1A0); no longer U2.1, U3.8 (1A3)
- net DMUX_5: now also U2.3, U3.4 (1A1); no longer U2.2, U3.6 (1A2)
- net DMUX_6: now also U2.2, U3.6 (1A2); no longer U2.3, U3.4 (1A1)
- net DMUX_7: now also U2.1, U3.8 (1A3); no longer U2.4, U3.2 (1A0)
Changed lines of the file:
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@@
 	)
 	(label "DMUX_6"
-		(at 205.74 115.57 0)
+		(at 205.74 118.11 0)
 		(effects
 			(font
@@
 	)
 	(label "DMUX_4"
-		(at 194.945 128.27 180)
+		(at 194.945 120.65 180)
 		(effects
 			(font
@@
 	)
 	(label "DMUX_5"
-		(at 205.74 118.11 0)
+		(at 205.74 115.57 0)
 		(effects
 			(font
@@
 	)
 	(label "DMUX_6"
-		(at 194.945 123.19 180)
+		(at 194.945 125.73 180)
 		(effects
 			(font
@@
 	)
 	(label "DMUX_7"
-		(at 205.74 113.03 0)
+		(at 205.74 120.65 0)
 		(effects
 			(font
@@
 	)
 	(label "DMUX_7"
-		(at 194.945 120.65 180)
+		(at 194.945 128.27 180)
 		(effects
 			(font
@@
 	)
 	(label "DMUX_5"
-		(at 194.945 125.73 180)
+		(at 194.945 123.19 180)
 		(effects
 			(font
@@
 	)
 	(label "DMUX_4"
-		(at 205.74 120.65 0)
-		(effects
-			(font
+		(at 205.74 113.03 0)
+		(effects
+			(font

Commit message: Updated connector on bo
Parts:
- renumbered D1 to D0, D2 to D1, D3 to D2, D4 to D3, D5 to D4, D6 to D5, D7 to D6, D8 to D7, SW1 to SW0, SW2 to SW1, SW3 to SW2, SW4 to SW3, SW5 to SW4, SW6 to SW5, SW7 to SW6, SW8 to SW7
Connections:
- net DMUX_0: no longer J2.16 (Pin_16)
- net DMUX_1: no longer J2.14 (Pin_14)
- net DMUX_2: no longer J2.12 (Pin_12)
- net DMUX_3: no longer J2.10 (Pin_10)
- net DMUX_4: no longer J2.8 (Pin_8)
- net DMUX_5: no longer J2.6 (Pin_6)
- net DMUX_6: no longer J2.4 (Pin_4)
- net DMUX_7: no longer J2.2 (Pin_2)
- no-connect marks 0 -> 8

Commit message: Corrected the pin connections of the playground
Parts:
- renumbered D7 to D0, D6 to D1, D5 to D2, D4 to D3, D3 to D4, D2 to D5, D1 to D6, D0 to D7, SW7 to SW0, SW6 to SW1, SW5 to SW2, SW4 to SW3, SW3 to SW4, SW2 to SW5, SW1 to SW6, SW0 to SW7
Connections:
- net DMUX_0: now also J2.1 (Pin_1), R8.1, SW0.1, U2.1, U3.8 (1A3); no longer J2.15 (Pin_15), R1.1, SW7.1, U1.4, U3.11 (2A3)
- net DMUX_1: now also J2.3 (Pin_3), R7.1, SW1.1, U2.2, U3.6 (1A2); no longer J2.13 (Pin_13), R2.1, SW6.1, U1.3, U3.13 (2A2)
- net DMUX_2: now also J2.5 (Pin_5), R6.1, SW2.1, U2.3, U3.4 (1A1); no longer J2.11 (Pin_11), R3.1, SW5.1, U1.2, U3.15 (2A1)
- net DMUX_3: now also J2.7 (Pin_7), R5.1, SW3.1, U2.4, U3.2 (1A0); no longer J2.9 (Pin_9), R4.1, SW4.1, U1.1, U3.17 (2A0)
- net DMUX_4: now also J2.9 (Pin_9), R4.1, SW4.1, U1.1, U3.17 (2A0); no longer J2.7 (Pin_7), R5.1, SW3.1, U2.4, U3.2 (1A0)
- net DMUX_5: now also J2.11 (Pin_11), R3.1, SW5.1, U1.2, U3.15 (2A1); no longer J2.5 (Pin_5), R6.1, SW2.1, U2.3, U3.4 (1A1)
- net DMUX_6: now also J2.13 (Pin_13), R2.1, SW6.1, U1.3, U3.13 (2A2); no longer J2.3 (Pin_3), R7.1, SW1.1, U2.2, U3.6 (1A2)
- net DMUX_7: now also J2.15 (Pin_15), R1.1, SW7.1, U1.4, U3.11 (2A3); no longer J2.1 (Pin_1), R8.1, SW0.1, U2.1, U3.8 (1A3)
- net at R13.1: now also U3.5 (2Y1); no longer U3.14 (1Y2)
- net at U3.12 (1Y3): now also R18.1; no longer R14.1
- net at U3.16 (1Y1): now also R16.1; no longer R12.1
- net at U3.18 (1Y0): now also R15.1; no longer R11.1
- net at U3.3 (2Y0): now also R14.1; no longer R15.1
- net at R17.1: now also U3.14 (1Y2); no longer U3.7 (2Y2)
- net at U3.9 (2Y3): now also R11.1; no longer R18.1
- new net: R12.1, U3.7 (2Y2)
Other:
- moved on the sheet: D0, D1, D2, D3, D4, D5, D6, D7, R11, R12, R13, R14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
