File: heepokranios-bo/heepokranios-bo.kicad_pcb (KiCad board)
At the start: 4 copper layers, 150.1 x 168.4 mm, 241 parts, among them IC1 ADA4945-1ACPZ-R7, IC2 ADA4945-1ACPZ-R7, IC3 ADA4945-1ACPZ-R7, IC4 ADA4945-1ACPZ-R7, IC5 ADA4945-1ACPZ-R7, J1 Conn_02x02_Odd_Even, J11 PGA_13x13, J14 Conn_02x03_Odd_Even, J15 Conn_02x08_Odd_Even, J16 Conn_02x03_Odd_Even, J17 Conn_02x03_Odd_Even, J18 Conn_01x03, J19 Conn_01x03, J2 Conn_02x02_Odd_Even, J20 Conn_01x03, J21 Conn_01x02, J22 Conn_01x03, J23 Conn_02x02_Odd_Even, J24 Conn_02x02_Odd_Even, J25 Conn_02x02_Odd_Even, J26 Conn_01x02, J27 Conn_01x02, J28 Conn_02x02_Odd_Even, J29 Conn_01x02, J3 Conn_02x03_Odd_Even, J30 Conn_01x02, J31 Conn_01x02, J32 Conn_01x02, J33 Conn_01x02, J34 Conn_01x02, J35 Conn_01x02, J36 Conn_01x02, J37 Conn_01x02, J38 Conn_01x02, J39 Conn_01x02, J4 Conn_02x03_Odd_Even, J40 Conn_01x02, J41 Conn_01x02, J42 Conn_01x02, J43 Conn_01x02, J44 Conn_02x02_Odd_Even, J45 Conn_01x03, J48 Conn_01x02, J49 Conn_01x02, J5 Conn_02x03_Odd_Even, J6 Conn_02x04_Odd_Even, J8 Conn_02x03_Odd_Even, J9 Conn_02x02_Odd_Even, SW1 SW_Push, U1 BIWIN_DTS04GE_SMD

Commit message: Changed NC pins to gnd connections of substrate as per the bonding diagram
Connections:
- J11 pad F11: unconnected-(J11-67-PadF11) -> GND
- J11 pad F2: unconnected-(J11-10-PadF2) -> GND
- J11 pad L7: unconnected-(J11-38-PadL7) -> GND
- J11 pad M10: unconnected-(J11-46-PadM10) -> GND
- J11 pad M11: unconnected-(J11-49-PadM11) -> GND
- J11 pad M9: unconnected-(J11-44-PadM9) -> GND
