File: heepokranios-bo/subsheets/fd_buffer.kicad_sch (KiCad schematic)
At the start: 17 parts, among them IC1 ADA4945-1ACPZ-R7, J18 Conn_01x03, J23 Conn_02x02_Odd_Even

Commit message: Changed in sch and board the fully diff amplifiers within the buffers to the THS4551IRGTR as there was no more stock of the one from Analog Devices
Parts:
- removed IC1: ADA4945-1ACPZ-R7, heepokranios-bo-library:QFN50P300X300X80-17N-D, symbol ADA4945-1ACPZ-R7:ADA4945-1ACPZ-R7
- added IC1: THS4551IRGTR, RGT0016C, symbol heepokranios-bo-library:THS4551IRGTR
Connections:
- net 3V3: now also IC1.12 (PD_N), IC1.5 (VS+), IC1.6 (VS+), IC1.7 (VS+), IC1.8 (VS+)
- net GND: now also IC1.13 (VS-), IC1.14 (VS-), IC1.15 (VS-), IC1.16 (VS-), IC1.17 (EP)
- net INT_OUT_N: now also IC1.11 (OUT-); no longer RF1.1
- net INT_OUT_P: now also IC1.10 (OUT+); no longer RF2.2
- net SEL_VCM: now also IC1.9 (VOCM)
- net at RF2.1, RG2.1: now also IC1.3 (IN-)
- net at RF1.2, RG1.1: now also IC1.2 (IN+)
- new net INT_FB_N: IC1.1 (FB-), RF1.1
- new net INT_FB_P: IC1.4 (FB+), RF2.2
Other:
- note added: "Not used in this version"
- note added: "Not used in this version Only provides 3V3 and GND"
- note removed: "Note: If not enough stock, can replace it for the THS4551, pinout will change!"
- note removed: "Short this for HP mode"
- note removed: "Short this for LP mode"
- moved on the sheet: C52, C53, C54, C55, C56, J18, J23, RF1, RF2, RG1, RG2
